File: Hardware/SparkFun_Pro_Micro.sch (EAGLE design)
At the start: 33 parts, among them U2 MIC5219, U3 ATMEGA32U4, Y1 16MHz

Commit message: Fixing 32u4 pin names
Connections:
- net D14: now also U3.PB3(MISO); no longer U3.PB0(SS)
- net MISO: now also U3.PB0(SS); no longer U3.PB3(MISO)
Changed lines of the file:
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@@
 <?xml version="1.0" encoding="utf-8"?>
 <!DOCTYPE eagle SYSTEM "eagle.dtd">
-<eagle version="6.4">
+<eagle version="7.3.0">
 <drawing>
 <settings>
@@
 <layer number="54" name="bGND_GNDA" color="1" fill="9" visible="no" active="no"/>
 <layer number="56" name="wert" color="7" fill="1" visible="no" active="no"/>
+<layer number="90" name="Modules" color="5" fill="1" visible="yes" active="yes"/>
 <layer number="91" name="Nets" color="2" fill="1" visible="yes" active="yes"/>
 <layer number="92" name="Busses" color="1" fill="1" visible="yes" active="yes"/>
@@
 <layer number="254" name="cooling" color="7" fill="1" visible="yes" active="yes"/>
 </layers>
-<schematic>
+<schematic xreflabel="%F%N/%S" xrefpart="/%S">
 <attributes>
 </attributes>
@@
 <wire x1="198.12" y1="91.44" x2="205.74" y2="91.44" width="0.1524" layer="91"/>
 <label x="200.66" y="91.44" size="1.778" layer="95"/>
-<pinref part="U3" gate="G$1" pin="PB3(MISO)"/>
+<pinref part="U3" gate="G$1" pin="PB0(SS)"/>
 </segment>
 </net>
@@
 <wire x1="210.82" y1="86.36" x2="210.82" y2="83.82" width="0.1524" layer="91"/>
 <label x="200.66" y="99.06" size="1.778" layer="95"/>
-<pinref part="U3" gate="G$1" pin="PB0(SS)"/>
+<pinref part="U3" gate="G$1" pin="PB3(MISO)"/>
 <pinref part="R4" gate="G$1" pin="1"/>
 </segment>

Commit message: Proto finished. Add ignore.
Parts:
- removed C13, C19: 10uF, SparkFun:CAP_POL1206
- removed JP6, JP7: M12PTH, SparkFun:M12PTH
- removed R5, R7: 22, SparkFun:RESISTOR0603-RES
- removed U$1: LOGO-SFESK, SparkFun:LOGO-SFESK
- removed U$11: LOGO-SFENEW, SparkFun:LOGO-SFENEW
- removed U2: MIC5219, SparkFun:V_REG_LDOSMD
- removed X1: (no value), Testing:USB-ABIN&OUT
- removed Y1: 16MHz, SparkFun:CRYSTAL5X3
- added C7, C8: 10uF, SparkFun-Capacitors:10UF-0603-6.3V-20%
- added J1: (no value), USBC:USB_C4
- added J2: Qwiic, SparkFun-Connectors:QWIIC_CONNECTORJS-1MM
- added J3, J4: (no value), Castellated:CONN_12CASTLE
- added LOGO1: SFE_LOGO_NAME_FLAME.1_INCH, SparkFun-Aesthetics:SFE_LOGO_NAME_FLAME.1_INCH
- added LOGO2: QWIIC_LOGO_4MM, SparkFun-Aesthetics:QWIIC_LOGO_4MM
- added LOGO3: QWIIC_LOGO_6MM, SparkFun-Aesthetics:QWIIC_LOGO_6MM
- added R1, R3: 5.1k, SparkFun-Resistors:5.1KOHM-0402T-1/16W-1%
- added R8, R9: 22, SparkFun-Resistors:22OHM-0402T-1/16W-1%
- added S1: Reset, SparkFun-Switches:MOMENTARY-SWITCH-SPST-SMD-4.6X2.8MM
- added U1: 3.3V, SparkFun-IC-Power:V_REG_AP2112K-3.3V
- added Y2: 32MHz, SparkFun-Clocks:CRYSTAL-32MHZ-SMD-2.0X1.6MM
- C1, C3: device SparkFun:CAP0603-CAP -> SparkFun-Capacitors:0.1UF-0402T-16V-10%
- C10, C5, C6: value 1uF -> 1.0uF; device SparkFun:CAP0603-CAP -> SparkFun-Capacitors:1.0UF-0402T-16V-10%
- C2, C4: device SparkFun:CAP0603-CAP -> SparkFun-Capacitors:22PF-0402T-16V-10%
- D1: device SparkFun:LED0603 -> SparkFun-LED:LED-YELLOW0603
- D2: value (none) -> 3A/10V/280mV; device SparkFun:DIODESOD -> SparkFun-DiscreteSemi:DIODE-SCHOTTKY-BAT60A
- D3: value Green -> GREEN; device SparkFun:LED0603 -> SparkFun-LED:LED-GREEN0603
- F1: value 500mA -> 6V 0.5A; device SparkFun:PTCSMD -> SparkFun-Fuses:PPTC_6V500MA
- JP1, JP2: value FIDUCIALUFIDUCIAL -> FIDUCIAL1X2; device SparkFun:FIDUCIALUFIDUCIAL -> SparkFun-Aesthetics:FIDUCIAL1X2
- LED1: value Red -> RED; device SparkFun:LED0603 -> SparkFun-LED:LED-RED0603
- R11: value 1K -> 1k; device SparkFun:RESISTOR0603-RES -> SparkFun-Resistors:1KOHM-0402T-1/16W-1%
- R2: value 10K -> 10k; device SparkFun:RESISTOR0603-RES -> SparkFun-Resistors:10KOHM-0402T-1/16W-1%
- R4, R6: value 330 -> 1k; device SparkFun:RESISTOR0603-RES -> SparkFun-Resistors:1KOHM-0402T-1/16W-1%
- SJ1: device SparkFun:SOLDERJUMPERNC -> SparkFun-Jumpers:JUMPER-SMT_2_NO_SILK
- U$3: value OSHW-LOGOS -> OSHW-LOGOMINI; device SparkFun:OSHW-LOGOS -> SparkFun-Aesthetics:OSHW-LOGOMINI
- U3: value ATMEGA32U4 -> ATmega32U4; device Testing:ATMEGA32U4OUTFAKES -> SparkFun-IC-Microcontroller:ATMEGA32U41:1
Connections:
- net N$3 renamed USB_RAW
- net N$4 renamed UCAP
- removed net A4: U3.PF1(ADC1)
- removed net A5: U3.PF0(ADC0)
- removed net D11: U3.PB7
- removed net D12: U3.PD6(ADC9)
- removed net D13: U3.PC7
- removed net D14: R4.1, U3.PB3(MISO)
- removed net D2: JP7.8, U3.PD1(SDA)
- removed net D3: JP7.7, U3.PD0(SCL)
- removed net N$6: R7.2, X1.D-
- removed net N$8: R5.2, X1.D+
- removed net UVCC: C6.2, F1.1, U3.UVCC, U3.VBUS, X1.VBUS
- new net D-_HV: J1.D-, R8.1
- new net D2/SDA: J2.3, J3.8, U3.PD1(SDA)
- new net D3/SCL: J2.4, J3.7, U3.PD0(SCL)
- new net DP_HV: J1.D+, R9.1
- new net N$10: J1.CC2, R1.2
- new net N$3: J3.10
- new net N$9: J1.CC1, R3.2
- new net RXLED: R4.1, U3.PB0(SS)
- new net V_USB: C6.2, F1.1, J1.VBUS, U3.UVCC, U3.VBUS
- net A0: now also J4.8; no longer JP6.8
- net A1: now also J4.7; no longer JP6.7
- net A2: now also J4.6; no longer JP6.6
- net A3: now also J4.5; no longer JP6.5
- net D+: now also R9.2; no longer R5.1
- net D-: now also R8.2; no longer R7.1
- net D10: now also J4.12; no longer JP6.12
- net D4: now also J3.6; no longer JP7.6
- net D5: now also J3.5; no longer JP7.5
- net D6: now also J3.4; no longer JP7.4
- net D7: now also J3.3; no longer JP7.3
- net D8: now also J3.2; no longer JP7.2
- net D9: now also J3.1; no longer JP7.1
- net GND: now also C10.1, C7.1, C8.1, J1.GND, J2.1, J3.9, J4.2, R1.1, R3.1, S1.1, U1.GND, U3.GND; no longer C10.2, C13.-, C19.-, JP6.2, JP7.10, JP7.9, U2.GND, U3.GND@15, U3.GND@23, U3.GND@35, U3.GND@43, U3.UGND, X1.GND
- net MISO: now also J4.10, U3.PB3(MISO); no longer JP6.10, U3.PB0(SS)
- net MOSI: now also J4.11; no longer JP6.11
- net N$1: now also Y2.1; no longer Y1.1
- net N$2: now also Y2.2; no longer Y1.2
- net RAW: now also C7.2, J4.1, U1.EN, U1.IN; no longer C19.+, JP6.1, U2.EN, U2.IN
- net RESET: now also J4.3, S1.2; no longer JP6.3
- net RXI: now also J3.11; no longer JP7.11
- net SCK: now also J4.9; no longer JP6.9
- net TXO: now also J3.12; no longer JP7.12
- net VCC: now also C10.2, C8.2, J2.2, J4.4, U1.OUT; no longer C10.1, C13.+, JP6.4, U2.OUT, U3.AVCC@44, U3.VCC@34
Other:
- note added: "Close jumper to run board at 5V"
- note added: "Max Current Output: 600mA"
- note added: "Max Voltage Input: 6VDC"
- note added: "v20"
- note removed: "Added fuse and diode protection"
- note removed: "Added two small squares of tRestrict to keep the ground plane away from the sides of IC legs"
- note removed: "Board is marked with combination of"
- note removed: "Change to 500mA regulator"
- note removed: "Changed LEDs to be tied to VCC"
- note removed: "Changes on v1.1:"
- note removed: "Changes on v1.2:"
- note removed: "Changes on v1.3:"
- note removed: "Corrected silk on D14"
- note removed: "Max Current Output: 500mA"
- note removed: "Max Voltage Input: 16VDC"
- note removed: "Not used"
- note removed: "Open for 3.3V Board"
- note removed: "Renamed SS net to D14 (from D17)"
- note removed: "Routed directly inward or outward from each leg on the IC"
- note removed: "Updated QFN package on 32U4 to be 1:1"
- note removed: "Updated package on USB micro B (2 new pads)"
- note removed: "Updated symbol of 32U4 in schematic (switched MISO and SS placement)"
- note removed: "VCC = 5V or 3.3V Output"
- note removed: "resonator frequency and regulator voltage."
- note removed: "v13"
- moved on the sheet: C1, C10, C2, C3, C4, C5, C6, R11, R2, R4, R6
