File: Hardware/SparkFun_Pro_Micro-FP.brd (EAGLE design)
At the start: 17.8 x 33 mm, 105 parts, among them J2 Qwiic, U1 3.3V, U3 ATmega32U4, Y2 32MHz

Commit message: Adding production panel, pro micro FP test brd, and castellated test lbr.
Parts:
- added U2: PRO_MICRO_C, Castellated:PRO_MICRO_C
Changed lines of the file:
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@@
 <setting verticaltext="up"/>
 </settings>
-<grid distance="0.05" unitdist="inch" unit="inch" style="lines" multiple="1" display="yes" altdistance="0.0025" altunitdist="inch" altunit="inch"/>
+<grid distance="0.05" unitdist="inch" unit="inch" style="lines" multiple="1" display="yes" altdistance="0.005" altunitdist="inch" altunit="inch"/>
 <layers>
 <layer number="1" name="Top" color="4" fill="1" visible="yes" active="yes"/>
@@
 <element name="U$65" library="buzzard_labels (10)" package="5V1" value="" x="14.732" y="20.066" smashed="yes" rot="R90"/>
 <element name="U$15" library="buzzard_labels (10)" package="5V1" value="" x="16.383" y="21.59" smashed="yes" rot="MR0"/>
+<element name="U2" library="Castellated" package="PRO_MICRO_C" value="PRO_MICRO_C" x="-15.24" y="16.51" smashed="yes"/>
 </elements>
 <signals>
